Commit message: [UNTESTED] Committing files to migrate development to hprtx3060

File: xarm_description/urdf/dual_xarm_device.urdf.xacro (robot description, xacro)
@@ -15,6 +15,6 @@
   <xacro:arg name="model1300_1" default="false"/>
   <xacro:arg name="model1300_2" default="false"/>
-  <xacro:arg name="dof_1" default="7"/>
-  <xacro:arg name="dof_2" default="7"/>
+  <xacro:arg name="dof_1" default="6"/>
+  <xacro:arg name="dof_2" default="6"/>
   <xacro:arg name="robot_ip_1" default=""/>
   <xacro:arg name="robot_ip_2" default=""/>
@@ -64,4 +64,5 @@
   <!-- load xarm device -->
   <xacro:include filename="$(find xarm_description)/urdf/xarm_device_macro.xacro" />
+  <xacro:include filename="$(find xarm_description)/urdf/rotary_table.urdf.xacro" />
   <xacro:xarm_device prefix="$(arg prefix_1)" hw_ns="$(arg hw_ns)" limited="$(arg limited)"
     effort_control="$(arg effort_control)" velocity_control="$(arg velocity_control)"
@@ -102,3 +103,8 @@
     baud_checkset="$(arg baud_checkset_2)" default_gripper_baud="$(arg default_gripper_baud_2)"
     model1300="$(arg model1300_2)" robot_sn="$(arg robot_sn_2)" mesh_suffix="$(arg mesh_suffix)" kinematics_suffix="$(arg kinematics_suffix_2)" />
+    <!-- <joint name="world_to_rotary_stand" type="fixed">
+      <parent link="world"/>
+      <child link="rotary_stand"/>
+      <origin xyz="0 0.5 0" rpy="0 0 0"/>
+    </joint> -->
 </robot>

File: xarm_description/urdf/xarm6/xarm6.urdf.xacro (robot description, xacro)
@@ -5,7 +5,7 @@
     joint2_lower_limit:=${-2.059}  joint2_upper_limit:=${2.0944}
     joint3_lower_limit:=${-3.927}  joint3_upper_limit:=${0.19198}
-    joint4_lower_limit:=${-2.0*pi}  joint4_upper_limit:=${2.0*pi}
+    joint4_lower_limit:=${-0.5*pi}  joint4_upper_limit:=${0.5*pi}
     joint5_lower_limit:=${-1.69297}  joint5_upper_limit:=${pi}
-    joint6_lower_limit:=${-2.0*pi}  joint6_upper_limit:=${2.0*pi}
+    joint6_lower_limit:=${-0.5*pi}  joint6_upper_limit:=${0.5*pi}
     model_num:=0
     inertial_params_filename:='' kinematics_params_filename:='' "

File: xarm_moveit_config/srdf/dual_xarm.srdf.xacro (robot description, xacro)
@@ -16,4 +16,5 @@
   <xacro:arg name="add_other_geometry_1" default="false" />
   <xacro:arg name="add_other_geometry_2" default="false" />
+  <!-- Include the per-arm macros -->
   <xacro:include filename="$(find xarm_moveit_config)/srdf/xarm_macro.srdf.xacro" />
   <xacro:xarm_macro_srdf prefix="$(arg prefix_1)" dof="$(arg dof_1)" robot_type="$(arg robot_type_1)"
@@ -21,3 +22,32 @@
   <xacro:xarm_macro_srdf prefix="$(arg prefix_2)" dof="$(arg dof_2)" robot_type="$(arg robot_type_2)"
     add_gripper="$(arg add_gripper_2)" add_vacuum_gripper="$(arg add_vacuum_gripper_2)" add_bio_gripper="$(arg add_bio_gripper_2)" add_other_geometry="$(arg add_other_geometry_2)" />
+  <!-- NEW: Add a combined group for both arms -->
+  <group name="dual_arm">
+    <chain base_link="$(arg prefix_1)link_base" tip_link="$(arg prefix_1)link6" />
+    <chain base_link="$(arg prefix_2)link_base" tip_link="$(arg prefix_2)link6" />
+  </group>
+  <!-- Optionally, you could be more explicit with joints instead of chain -->
+  <group name="dual_arm">
+    <joint name="$(arg prefix_1)joint1"/>
+    <joint name="$(arg prefix_1)joint2"/>
+    <joint name="$(arg prefix_1)joint3"/>
+    <joint name="$(arg prefix_1)joint4"/>
+    <joint name="$(arg prefix_1)joint5"/>
+    <joint name="$(arg prefix_1)joint6"/>
+    <!-- <joint name="$(arg prefix_1)joint7"/> -->
+    <joint name="$(arg prefix_2)joint1"/>
+    <joint name="$(arg prefix_2)joint2"/>
+    <joint name="$(arg prefix_2)joint3"/>
+    <joint name="$(arg prefix_2)joint4"/>
+    <joint name="$(arg prefix_2)joint5"/>
+    <joint name="$(arg prefix_2)joint6"/>
+    <!-- <joint name="$(arg prefix_2)joint7"/> -->
+  </group>
+<group name="rotary_table">
+  <joint name="rotary_table_joint"/>
+</group>
+<group name="dual_arm_with_table">
+  <group name="dual_arm"/>
+  <group name="rotary_table"/>
+</group>
 </robot>

Commit message: [DELETE] Removed commenetd out section

File: xarm_description/urdf/dual_xarm_device.urdf.xacro (robot description, xacro)
@@ -103,8 +103,3 @@
     baud_checkset="$(arg baud_checkset_2)" default_gripper_baud="$(arg default_gripper_baud_2)"
     model1300="$(arg model1300_2)" robot_sn="$(arg robot_sn_2)" mesh_suffix="$(arg mesh_suffix)" kinematics_suffix="$(arg kinematics_suffix_2)" />
-    <!-- <joint name="world_to_rotary_stand" type="fixed">
-      <parent link="world"/>
-      <child link="rotary_stand"/>
-      <origin xyz="0 0.5 0" rpy="0 0 0"/>
-    </joint> -->
 </robot>
