Commit message: Update xarm_description/urdf/rotary_table.urdf.xacro
Co-authored-by: Copilot <175728472+Copilot@users.noreply.github.com>

File: xarm_description/urdf/rotary_table.urdf.xacro (robot description, xacro)
@@ -6,5 +6,5 @@
       <origin xyz="-0.200 0.200 0" rpy="1.5708 0 0"/>
       <geometry>
-        <mesh filename="file:///home/hprtx3060/xarm_ws_humble/src/xarm_ros2_fork/xarm_moveit_config/meshes/rotary_stand_m.STL" scale="1 1 1"/>
+        <mesh filename="package://xarm_moveit_config/meshes/rotary_stand_m.STL" scale="1 1 1"/>
       </geometry>
     </visual>
@@ -12,5 +12,5 @@
       <origin xyz="-0.200 0.200 0" rpy="1.5708 0 0"/>
       <geometry>
-        <mesh filename="file:///home/hprtx3060/xarm_ws_humble/src/xarm_ros2_fork/xarm_moveit_config/meshes/rotary_stand_m.STL" scale="1 1 1"/>
+        <mesh filename="package://xarm_moveit_config/meshes/rotary_stand_m.STL" scale="1 1 1"/>
       </geometry>
     </collision>

Commit message: Update xarm_description/urdf/rotary_table.urdf.xacro
Co-authored-by: Copilot <175728472+Copilot@users.noreply.github.com>

File: xarm_description/urdf/rotary_table.urdf.xacro (robot description, xacro)
@@ -20,5 +20,5 @@
       <origin xyz="-0.200 0.200 0.18" rpy="1.5708 0 0"/>
       <geometry>
-        <mesh filename="file:///home/hprtx3060/xarm_ws_humble/src/xarm_ros2_fork/xarm_moveit_config/meshes/RotaryPlate_m.STL" scale="1 1 1"/>
+        <mesh filename="package://xarm_moveit_config/meshes/RotaryPlate_m.STL" scale="1 1 1"/>
       </geometry>
     </visual>
@@ -26,5 +26,5 @@
       <origin xyz="-0.200 0.200 0.18" rpy="1.5708 0 0"/>
       <geometry>
-        <mesh filename="file:///home/hprtx3060/xarm_ws_humble/src/xarm_ros2_fork/xarm_moveit_config/meshes/RotaryPlate_m.STL" scale="1 1 1"/>
+        <mesh filename="package://xarm_moveit_config/meshes/RotaryPlate_m.STL" scale="1 1 1"/>
       </geometry>
     </collision>
