Commit message: [ADD] Integrated rotary table with xarm

File: xarm_description/urdf/rotary_table.urdf.xacro (robot description, xacro)
@@ -6,5 +6,5 @@
       <origin xyz="-0.200 0.200 0" rpy="1.5708 0 0"/>
       <geometry>
-        <mesh filename="file:///home/dellubuntu/xarm_ws_humble/src/xarm_ros2_fork/xarm_moveit_config/meshes/rotary_stand_m.STL" scale="1 1 1"/>
+        <mesh filename="file:///home/hprtx3060/xarm_ws_humble/src/xarm_ros2_fork/xarm_moveit_config/meshes/rotary_stand_m.STL" scale="1 1 1"/>
       </geometry>
     </visual>
@@ -12,5 +12,5 @@
       <origin xyz="-0.200 0.200 0" rpy="1.5708 0 0"/>
       <geometry>
-        <mesh filename="file:///home/dellubuntu/xarm_ws_humble/src/xarm_ros2_fork/xarm_moveit_config/meshes/rotary_stand_m.STL" scale="1 1 1"/>
+        <mesh filename="file:///home/hprtx3060/xarm_ws_humble/src/xarm_ros2_fork/xarm_moveit_config/meshes/rotary_stand_m.STL" scale="1 1 1"/>
       </geometry>
     </collision>
@@ -20,5 +20,5 @@
       <origin xyz="-0.200 0.200 0.18" rpy="1.5708 0 0"/>
       <geometry>
-        <mesh filename="file:///home/dellubuntu/xarm_ws_humble/src/xarm_ros2_fork/xarm_moveit_config/meshes/RotaryPlate_m.STL" scale="1 1 1"/>
+        <mesh filename="file:///home/hprtx3060/xarm_ws_humble/src/xarm_ros2_fork/xarm_moveit_config/meshes/RotaryPlate_m.STL" scale="1 1 1"/>
       </geometry>
     </visual>
@@ -26,5 +26,5 @@
       <origin xyz="-0.200 0.200 0.18" rpy="1.5708 0 0"/>
       <geometry>
-        <mesh filename="file:///home/dellubuntu/xarm_ws_humble/src/xarm_ros2_fork/xarm_moveit_config/meshes/RotaryPlate_m.STL" scale="1 1 1"/>
+        <mesh filename="file:///home/hprtx3060/xarm_ws_humble/src/xarm_ros2_fork/xarm_moveit_config/meshes/RotaryPlate_m.STL" scale="1 1 1"/>
       </geometry>
     </collision>

File: xarm_description/urdf/xarm_device.urdf.xacro (robot description, xacro)
@@ -1,4 +1,10 @@
-<?xml version='1.0' encoding='utf-8'?>
+<?xml version="1.0" encoding="utf-8"?>
+<!--
+  Single xArm device + independent simulated rotary table.
+  The xArm block is unchanged from the original template. A second
+  kinematic chain (rotary table) is added and connected to <world>.
+-->
 <robot xmlns:xacro="http://ros.org/wiki/xacro" name="UF_ROBOT">
+  <!-- ‣‣‣ Existing xArm argument list (unchanged) -->
   <xacro:arg name="prefix" default=""/>
   <xacro:arg name="hw_ns" default="xarm"/>
@@ -10,5 +16,5 @@
   <xacro:arg name="add_bio_gripper" default="false"/>
   <xacro:arg name="model1300" default="false"/>
-  <xacro:arg name="dof" default="7"/>
+  <xacro:arg name="dof" default="6"/>
   <xacro:arg name="robot_ip" default=""/>
   <xacro:arg name="robot_type" default="xarm"/>
@@ -39,5 +45,11 @@
   <xacro:arg name="mesh_suffix" default="stl"/>
   <xacro:arg name="kinematics_suffix" default=""/>
-  <!-- load xarm device -->
+  <!-- ‣‣‣ NEW parameters for the rotary table -->
+  <xacro:property name="rot_base_radius" value="0.20"/>
+  <xacro:property name="rot_base_height" value="0.18"/>
+  <xacro:property name="rot_plate_radius" value="0.20"/>
+  <xacro:property name="rot_plate_height" value="0.18"/>
+  <xacro:property name="rot_origin_xyz" value="0 0.5 0"/>  <!-- position in world -->
+  <!-- ‣‣‣ xArm include (unchanged) -->
   <xacro:include filename="$(find xarm_description)/urdf/xarm_device_macro.xacro" />
   <xacro:xarm_device prefix="$(arg prefix)" hw_ns="$(arg hw_ns)" limited="$(arg limited)"
@@ -59,4 +71,87 @@
     baud_checkset="$(arg baud_checkset)" default_gripper_baud="$(arg default_gripper_baud)"
     model1300="$(arg model1300)" attach_to="$(arg attach_to)" attach_xyz="$(arg attach_xyz)" attach_rpy="$(arg attach_rpy)"
-    robot_sn="$(arg robot_sn)" use_gazebo_camera="$(arg use_gazebo_camera)" mesh_suffix="$(arg mesh_suffix)" kinematics_suffix="$(arg kinematics_suffix)" />
+    robot_sn="$(arg robot_sn)" use_gazebo_camera="$(arg use_gazebo_camera)"
+    mesh_suffix="$(arg mesh_suffix)" kinematics_suffix="$(arg kinematics_suffix)" />
+  <!-- ‣‣‣ Independent rotary table kinematic chain -->
+  <link name="rotary_table_base">
+    <visual>
+      <origin xyz="0 0 0" rpy="1.5708 0 0"/>
+      <geometry>
+        <!-- <cylinder radius="${rot_base_radius}" length="${rot_base_height}"/> -->
+        <mesh filename="package://xarm_moveit_config/meshes/rotary_stand_centered.STL" />
+      </geometry>
+      <material name="RotaryGrey">
+        <color rgba="0.6 0.6 0.6 1"/>
+      </material>
+    </visual>
+    <collision>
+      <origin xyz="0 0 0" rpy="1.5708 0 0"/>
+      <geometry>
+        <!-- <cylinder radius="${rot_base_radius}" length="${rot_base_height}"/> -->
+        <mesh filename="package://xarm_moveit_config/meshes/rotary_stand_centered.STL" />
+      </geometry>
+    </collision>
+    <inertial>
+      <origin xyz="0 0 0" rpy="1.5708 0 0"/>
+      <mass value="5.0"/>
+      <inertia ixx="0.1" iyy="0.1" izz="0.1" ixy="0" ixz="0" iyz="0"/>
+    </inertial>
+  </link>
+  <!-- fixed transform world → rotary_table_base -->
+  <joint name="world_to_rotary_base" type="fixed">
+    <parent link="world"/>
+    <child  link="rotary_table_base"/>
+    <origin xyz="${rot_origin_xyz}" rpy="0 0 0"/>
+  </joint>
+  <!-- rotating plate -->
+  <link name="rotary_table_plate">
+    <visual>
+      <origin xyz="0 0 0" rpy="1.5708 0 0"/>
+      <geometry>
+        <!-- <cylinder radius="${rot_plate_radius}" length="${rot_plate_height}"/> -->
+        <mesh filename="package://xarm_moveit_config/meshes/RotaryPlate_centered.STL" />
+      </geometry>
+      <material name="RotaryBlue">
+        <color rgba="0.2 0.4 0.8 1"/>
+      </material>
+    </visual>
+    <collision>
+      <origin xyz="0 0 0" rpy="1.5708 0 0"/>
+      <geometry>
+        <mesh filename="package://xarm_moveit_config/meshes/RotaryPlate_centered.STL" />
+      </geometry>
+    </collision>
+    <inertial>
+      <origin xyz="0 0 0" rpy="1.5708 0 0"/>
+      <mass value="2.0"/>
+      <inertia ixx="0.02" iyy="0.02" izz="0.02" ixy="0" ixz="0" iyz="0"/>
+    </inertial>
+  </link>
+  <joint name="rotary_table_joint" type="revolute">
+    <parent link="rotary_table_base"/>
+    <child  link="rotary_table_plate"/>
+    <origin xyz="0 0 ${rot_base_height}" rpy="0 0 0"/>
+    <axis xyz="0 0 1"/>
+    <limit lower="-3.14159" upper="3.14159" effort="20" velocity="1.5"/>
+  </joint>
+  <!-- ros2_control specification for the rotary joint (fake hardware) -->
+  <ros2_control name="RotaryTableHW" type="system">
+    <hardware>
+      <plugin>mock_components/GenericSystem</plugin>
+      <!-- Either style below works →  pick one and keep it consistent -->
+      <!-- YAML-list style -->
+      <!-- <param name="joints">['rotary_table_joint']</param> -->
+      <!-- <param name="command_interfaces">['position']</param> -->
+      <!-- <param name="state_interfaces">['position']</param> -->
+      <!-- Plain space-separated style (simplest) -->
+      <param name="joints">rotary_table_joint</param>
+      <param name="command_interfaces">position</param>
+      <param name="state_interfaces">position</param>
+      <param name="fake_sensor_commands">true</param>
+    </hardware>
+    <joint name="rotary_table_joint">
+      <state_interface   name="position"/>
+      <command_interface name="position"/>
+    </joint>
+  </ros2_control>
 </robot>

Commit message: [ADD] RVIZ now reads table position

File: xarm_description/urdf/rotary_table.urdf.xacro (robot description, xacro)
@@ -33,5 +33,5 @@
     <parent link="world"/>
     <child link="rotary_stand"/>
-    <origin xyz="0 0.5 0" rpy="0 0 0"/>
+    <origin xyz="0.4915 -0.238 0" rpy="0 0 0"/>
   </joint>
   <joint name="rotary_table_joint" type="revolute">

File: xarm_description/urdf/xarm_device.urdf.xacro (robot description, xacro)
@@ -50,5 +50,5 @@
   <xacro:property name="rot_plate_radius" value="0.20"/>
   <xacro:property name="rot_plate_height" value="0.18"/>
-  <xacro:property name="rot_origin_xyz" value="0 0.5 0"/>  <!-- position in world -->
+  <xacro:property name="rot_origin_xyz" value="0.4915 -0.238 0"/>  <!-- position in world -->
   <!-- ‣‣‣ xArm include (unchanged) -->
   <xacro:include filename="$(find xarm_description)/urdf/xarm_device_macro.xacro" />

Commit message: [ADD] Added TF publisher to the pipeline

File: xarm_description/urdf/rotary_table.urdf.xacro (robot description, xacro)
@@ -2,5 +2,5 @@
 <robot xmlns:xacro="http://ros.org/wiki/xacro" name="rotary_table">
   <link name="world"/>
-  <link name="rotary_stand">
+  <link name="rotary_table_base">
     <visual>
       <origin xyz="-0.200 0.200 0" rpy="1.5708 0 0"/>
@@ -32,9 +32,9 @@
   <joint name="world_to_rotary_stand" type="fixed">
     <parent link="world"/>
-    <child link="rotary_stand"/>
+    <child link="rotary_table_base"/>
     <origin xyz="0.4915 -0.238 0" rpy="0 0 0"/>
   </joint>
   <joint name="rotary_table_joint" type="revolute">
-    <parent link="rotary_stand"/>
+    <parent link="rotary_table_base"/>
     <child link="rotary_plate"/>
     <origin xyz="0 0 0" rpy="0 0 0"/>

File: xarm_description/urdf/single_xarm_with_rotary.urdf.xacro (robot description, xacro)
@@ -58,8 +58,8 @@
     model1300="$(arg model1300)" robot_sn="$(arg robot_sn)"
     mesh_suffix="$(arg mesh_suffix)" kinematics_suffix="$(arg kinematics_suffix)" />
-  <joint name="world_to_rotary_stand" type="fixed">
+  <!-- <joint name="world_to_rotary_stand" type="fixed">
     <parent link="world"/>
     <child link="rotary_stand"/>
     <origin xyz="0 0.5 0" rpy="0 0 0"/>
-  </joint>
+  </joint> -->
 </robot>
