Commit message: [FIX] Fixed URDF structure

File: xarm_description/urdf/rotary_table.urdf.xacro (robot description, xacro)
@@ -1,64 +1,81 @@
 <?xml version="1.0"?>
 <robot xmlns:xacro="http://ros.org/wiki/xacro" name="rotary_table">
-  <link name="world"/>
+    <!-- ‣‣‣ NEW parameters for the rotary table -->
+  <xacro:property name="rot_base_radius" value="0.20"/>
+  <xacro:property name="rot_base_height" value="0.18"/>
+  <xacro:property name="rot_plate_radius" value="0.20"/>
+  <xacro:property name="rot_plate_height" value="0.188"/>
+  <xacro:property name="rot_origin_xyz" value="0.4915 -0.238 0"/>  <!-- position in world -->
   <link name="rotary_table_base">
     <visual>
-      <origin xyz="-0.200 0.200 0" rpy="1.5708 0 0"/>
+      <origin xyz="0 0 0" rpy="1.5708 0 0"/>
       <geometry>
-        <mesh filename="package://xarm_moveit_config/meshes/rotary_stand_m.STL" scale="1 1 1"/>
+        <mesh filename="package://xarm_moveit_config/meshes/rotary_stand_centered.STL" />
       </geometry>
+      <material name="RotaryGrey">
+        <color rgba="0.6 0.6 0.6 1"/>
+      </material>
     </visual>
     <collision>
-      <origin xyz="-0.200 0.200 0" rpy="1.5708 0 0"/>
+      <origin xyz="0 0 0" rpy="1.5708 0 0"/>
       <geometry>
-        <mesh filename="package://xarm_moveit_config/meshes/rotary_stand_m.STL" scale="1 1 1"/>
+        <mesh filename="package://xarm_moveit_config/meshes/rotary_stand_centered.STL" />
       </geometry>
     </collision>
+    <inertial>
+      <origin xyz="0 0 0" rpy="1.5708 0 0"/>
+      <mass value="5.0"/>
+      <inertia ixx="0.1" iyy="0.1" izz="0.1" ixy="0" ixz="0" iyz="0"/>
+    </inertial>
   </link>
-  <link name="rotary_plate">
+  <!-- fixed transform world → rotary_table_base -->
+  <joint name="world_to_rotary_base" type="fixed">
+    <parent link="world"/>
+    <child  link="rotary_table_base"/>
+    <origin xyz="${rot_origin_xyz}" rpy="0 0 0"/>
+  </joint>
+  <!-- rotating plate -->
+  <link name="rotary_table_plate">
     <visual>
-      <origin xyz="-0.200 0.200 0.18" rpy="1.5708 0 0"/>
+      <origin xyz="0 0 -0.008" rpy="1.5708 0 0"/>
       <geometry>
-        <mesh filename="package://xarm_moveit_config/meshes/RotaryPlate_m.STL" scale="1 1 1"/>
+        <!-- <cylinder radius="${rot_plate_radius}" length="${rot_plate_height}"/> -->
+        <mesh filename="package://xarm_moveit_config/meshes/RotaryPlate_centered.STL" />
       </geometry>
+      <material name="RotaryBlue">
+        <color rgba="0.2 0.4 0.8 1"/>
+      </material>
     </visual>
     <collision>
-      <origin xyz="-0.200 0.200 0.18" rpy="1.5708 0 0"/>
+      <origin xyz="0 0 -0.008" rpy="1.5708 0 0"/>
       <geometry>
-        <mesh filename="package://xarm_moveit_config/meshes/RotaryPlate_m.STL" scale="1 1 1"/>
+        <mesh filename="package://xarm_moveit_config/meshes/RotaryPlate_centered.STL" />
       </geometry>
     </collision>
+    <inertial>
+      <origin xyz="0 0 -0.008" rpy="1.5708 0 0"/>
+      <mass value="2.0"/>
+      <inertia ixx="0.02" iyy="0.02" izz="0.02" ixy="0" ixz="0" iyz="0"/>
+    </inertial>
   </link>
-  <joint name="world_to_rotary_stand" type="fixed">
-    <parent link="world"/>
-    <child link="rotary_table_base"/>
-    <origin xyz="0.4915 -0.238 0" rpy="0 0 0"/>
-  </joint>
   <joint name="rotary_table_joint" type="revolute">
     <parent link="rotary_table_base"/>
-    <child link="rotary_plate"/>
-    <origin xyz="0 0 0" rpy="0 0 0"/>
+    <child  link="rotary_table_plate"/>
+    <origin xyz="0 0 ${rot_base_height}" rpy="0 0 0"/>
     <axis xyz="0 0 1"/>
-    <limit lower="-3.14" upper="3.14" effort="10" velocity="1.0"/>
+    <limit lower="-3.14159" upper="3.14159" effort="20" velocity="1.5"/>
   </joint>
-  <transmission name="rotary_table_transmission">
-    <type>transmission_interface/SimpleTransmission</type>
-    <joint name="rotary_table_joint">
-      <hardwareInterface>hardware_interface/PositionJointInterface</hardwareInterface>
-    </joint>
-    <actuator name="rotary_table_motor">
-      <hardwareInterface>hardware_interface/PositionJointInterface</hardwareInterface>
-      <mechanicalReduction>1.0</mechanicalReduction>
-    </actuator>
-  </transmission>
+  <!-- ros2_control specification for the rotary joint (fake hardware) -->
   <ros2_control name="RotaryTableHW" type="system">
     <hardware>
       <plugin>mock_components/GenericSystem</plugin>
-      <param name="example_param_hw_start_duration">0.0</param>
-      <param name="example_param_hw_stop_duration">0.0</param>
-      <param name="example_param_hw_slowdown">1.0</param>
+      <!-- Plain space-separated style (simplest) -->
+      <param name="joints">rotary_table_joint</param>
+      <param name="command_interfaces">position</param>
+      <param name="state_interfaces">position</param>
+      <param name="fake_sensor_commands">true</param>
     </hardware>
     <joint name="rotary_table_joint">
-      <state_interface name="position"/>
+      <state_interface   name="position"/>
       <command_interface name="position"/>
     </joint>

File: xarm_description/urdf/single_xarm_with_rotary.urdf.xacro (robot description, xacro)
@@ -30,10 +30,17 @@
   <xacro:arg name="geometry_mesh_tcp_xyz" default="0 0 0"/>
   <xacro:arg name="geometry_mesh_tcp_rpy" default="0 0 0"/>
+  <xacro:arg name="add_walls" default="true"/>
   <xacro:arg name="baud_checkset" default="true"/>
   <xacro:arg name="default_gripper_baud" default="2000000"/>
   <xacro:arg name="mesh_suffix" default="stl"/>
   <xacro:arg name="kinematics_suffix" default=""/>
+  <xacro:arg name="attach_to" default="xarm_base"/>
+  <xacro:arg name="attach_xyz" default="0 0 0"/>
+  <xacro:arg name="attach_rpy" default="0 0 0"/>
+  <!-- <xacro:include filename="$(find xarm_description)/urdf/workcell_walls.urdf.xacro" /> -->
+  <xacro:include filename="$(find xarm_description)/urdf/cobot_environment_macro.xacro" />
   <xacro:include filename="$(find xarm_description)/urdf/xarm_device_macro.xacro"/>
   <xacro:include filename="$(find xarm_description)/urdf/rotary_table.urdf.xacro"/>
+  <xacro:cobot_environment add_walls="$(arg add_walls)" />
   <xacro:xarm_device prefix="" hw_ns="$(arg hw_ns)" limited="$(arg limited)"
     effort_control="$(arg effort_control)" velocity_control="$(arg velocity_control)"
@@ -42,5 +49,4 @@
     ros2_control_plugin="$(arg ros2_control_plugin)" robot_type="$(arg robot_type)"
     load_gazebo_plugin="false" ros2_control_params="$(arg ros2_control_params)"
-    attach_to="rotary_plate" attach_xyz="0 0 0" attach_rpy="0 0 0"
     add_realsense_d435i="$(arg add_realsense_d435i)"
     add_d435i_links="$(arg add_d435i_links)"
@@ -57,9 +63,5 @@
     baud_checkset="$(arg baud_checkset)" default_gripper_baud="$(arg default_gripper_baud)"
     model1300="$(arg model1300)" robot_sn="$(arg robot_sn)"
-    mesh_suffix="$(arg mesh_suffix)" kinematics_suffix="$(arg kinematics_suffix)" />
-  <!-- <joint name="world_to_rotary_stand" type="fixed">
-    <parent link="world"/>
-    <child link="rotary_stand"/>
-    <origin xyz="0 0.5 0" rpy="0 0 0"/>
-  </joint> -->
-</robot>
+    mesh_suffix="$(arg mesh_suffix)" kinematics_suffix="$(arg kinematics_suffix)"
+    attach_to="$(arg attach_to)" attach_xyz="$(arg attach_xyz)" attach_rpy="$(arg attach_rpy)"/>
+ </robot>

File: xarm_description/urdf/workcell_static_objects.urdf.xacro (robot description, xacro)
@@ -1,6 +1,29 @@
 <?xml version="1.0"?>
-<robot xmlns:xacro="http://ros.org/wiki/xacro" name="workcell_walls">
-  <xacro:macro name="workcell_walls" params="prefix:=''">
-    <link name="${prefix}floor">
+<robot xmlns:xacro="http://ros.org/wiki/xacro" name="workcell_static">
+  <xacro:macro name="workcell_static">
+<link name="world" />
+<link name="xarm_base">
+    <visual>
+      <origin xyz="0 0 -0.008" rpy="-3.14 0 -3.14"/>
+      <geometry>
+        <mesh filename="package://xarm_description/meshes/other/robot_base_m.STL" />
+      </geometry>
+      <material name="RotaryGrey">
+        <color rgba="0.6 0.6 0.6 1"/>
+      </material>
+    </visual>
+    <collision>
+      <origin xyz="0 0 -0.008" rpy="-3.14 0 -3.14"/>
+      <geometry>
+        <mesh filename="package://xarm_description/meshes/other/robot_base_m.STL" />
+      </geometry>
+    </collision>
+    <inertial>
+      <origin xyz="0 0 -0.008" rpy="-3.14 0 -3.14"/>
+      <mass value="5.0"/>
+      <inertia ixx="0.1" iyy="0.1" izz="0.1" ixy="0" ixz="0" iyz="0"/>
+    </inertial>
+  </link>
+    <link name="floor">
       <visual>
         <origin xyz="0 0 0" rpy="0 0 0"/>
@@ -19,5 +42,5 @@
       </collision>
     </link>
-    <link name="${prefix}back_wall">
+    <link name="back_wall">
       <visual>
         <origin xyz="0 0 0" rpy="0 0 0"/>
@@ -36,5 +59,5 @@
       </collision>
     </link>
-    <link name="${prefix}left_wall">
+    <link name="left_wall">
       <visual>
         <origin xyz="0 0 0" rpy="0 0 0"/>
@@ -53,5 +76,5 @@
       </collision>
     </link>
-    <link name="${prefix}right_wall">
+    <link name="right_wall">
       <visual>
         <origin xyz="0 0 0" rpy="0 0 0"/>

File: xarm_description/urdf/xarm_device.urdf.xacro (robot description, xacro)
@@ -38,5 +38,4 @@
   <xacro:arg name="geometry_mesh_tcp_xyz" default="0 0 0"/>
   <xacro:arg name="geometry_mesh_tcp_rpy" default="0 0 0"/>
-  <xacro:arg name="add_walls" default="false"/>
   <xacro:arg name="baud_checkset" default="true"/>
   <xacro:arg name="default_gripper_baud" default="2000000"/>
@@ -46,13 +45,7 @@
   <xacro:arg name="mesh_suffix" default="stl"/>
   <xacro:arg name="kinematics_suffix" default=""/>
-  <!-- ‣‣‣ NEW parameters for the rotary table -->
-  <xacro:property name="rot_base_radius" value="0.20"/>
-  <xacro:property name="rot_base_height" value="0.18"/>
-  <xacro:property name="rot_plate_radius" value="0.20"/>
-  <xacro:property name="rot_plate_height" value="0.18"/>
-  <xacro:property name="rot_origin_xyz" value="0.4915 -0.238 0"/>  <!-- position in world -->
   <!-- ‣‣‣ xArm include (unchanged) -->
   <xacro:include filename="$(find xarm_description)/urdf/xarm_device_macro.xacro" />
-  <xacro:include filename="$(find xarm_description)/urdf/workcell_walls.urdf.xacro" />
+  <!-- ‣‣‣ xArm device macro (unchanged) -->
   <xacro:xarm_device prefix="$(arg prefix)" hw_ns="$(arg hw_ns)" limited="$(arg limited)"
     effort_control="$(arg effort_control)" velocity_control="$(arg velocity_control)"
@@ -75,108 +68,3 @@
     robot_sn="$(arg robot_sn)" use_gazebo_camera="$(arg use_gazebo_camera)"
     mesh_suffix="$(arg mesh_suffix)" kinematics_suffix="$(arg kinematics_suffix)" />
-  <!-- ‣‣‣ Independent rotary table kinematic chain -->
-  <link name="rotary_table_base">
-    <visual>
-      <origin xyz="0 0 0" rpy="1.5708 0 0"/>
-      <geometry>
-        <!-- <cylinder radius="${rot_base_radius}" length="${rot_base_height}"/> -->
-        <mesh filename="package://xarm_moveit_config/meshes/rotary_stand_centered.STL" />
-      </geometry>
-      <material name="RotaryGrey">
-        <color rgba="0.6 0.6 0.6 1"/>
-      </material>
-    </visual>
-    <collision>
-      <origin xyz="0 0 0" rpy="1.5708 0 0"/>
-      <geometry>
-        <!-- <cylinder radius="${rot_base_radius}" length="${rot_base_height}"/> -->
-        <mesh filename="package://xarm_moveit_config/meshes/rotary_stand_centered.STL" />
-      </geometry>
-    </collision>
-    <inertial>
-      <origin xyz="0 0 0" rpy="1.5708 0 0"/>
-      <mass value="5.0"/>
-      <inertia ixx="0.1" iyy="0.1" izz="0.1" ixy="0" ixz="0" iyz="0"/>
-    </inertial>
-  </link>
-  <!-- fixed transform world → rotary_table_base -->
-  <joint name="world_to_rotary_base" type="fixed">
-    <parent link="world"/>
-    <child  link="rotary_table_base"/>
-    <origin xyz="${rot_origin_xyz}" rpy="0 0 0"/>
-  </joint>
-  <!-- rotating plate -->
-  <link name="rotary_table_plate">
-    <visual>
-      <origin xyz="0 0 0" rpy="1.5708 0 0"/>
-      <geometry>
-        <!-- <cylinder radius="${rot_plate_radius}" length="${rot_plate_height}"/> -->
-        <mesh filename="package://xarm_moveit_config/meshes/RotaryPlate_centered.STL" />
-      </geometry>
-      <material name="RotaryBlue">
-        <color rgba="0.2 0.4 0.8 1"/>
-      </material>
-    </visual>
-    <collision>
-      <origin xyz="0 0 0" rpy="1.5708 0 0"/>
-      <geometry>
-        <mesh filename="package://xarm_moveit_config/meshes/RotaryPlate_centered.STL" />
-      </geometry>
-    </collision>
-    <inertial>
-      <origin xyz="0 0 0" rpy="1.5708 0 0"/>
-      <mass value="2.0"/>
-      <inertia ixx="0.02" iyy="0.02" izz="0.02" ixy="0" ixz="0" iyz="0"/>
-    </inertial>
-  </link>
-  <joint name="rotary_table_joint" type="revolute">
-    <parent link="rotary_table_base"/>
-    <child  link="rotary_table_plate"/>
-    <origin xyz="0 0 ${rot_base_height}" rpy="0 0 0"/>
-    <axis xyz="0 0 1"/>
-    <limit lower="-3.14159" upper="3.14159" effort="20" velocity="1.5"/>
-  </joint>
-  <xacro:if value="${add_walls}">
-    <xacro:workcell_walls/>
-    <joint name="floor_joint" type="fixed">
-      <parent link="world"/>
-      <child  link="floor"/>
-      <origin xyz="0.355 -0.205 -0.0025" rpy="0 0 0"/>
-    </joint>
-    <joint name="back_wall_joint" type="fixed">
-      <parent link="world"/>
-      <child  link="back_wall"/>
-      <origin xyz="0.3825 0.5425 0.75" rpy="0 0 0"/>
-    </joint>
-    <joint name="left_wall_joint" type="fixed">
-      <parent link="world"/>
-      <child  link="left_wall"/>
-      <origin xyz="-0.4225 -0.2125 0.75" rpy="0 0 0"/>
-    </joint>
-    <joint name="right_wall_joint" type="fixed">
-      <parent link="world"/>
-      <child  link="right_wall"/>
-      <origin xyz="1.3375 -0.2125 0.75" rpy="0 0 0"/>
-    </joint>
-  </xacro:if>
-  <!-- ros2_control specification for the rotary joint (fake hardware) -->
-  <ros2_control name="RotaryTableHW" type="system">
-    <hardware>
-      <plugin>mock_components/GenericSystem</plugin>
-      <!-- Either style below works →  pick one and keep it consistent -->
-      <!-- YAML-list style -->
-      <!-- <param name="joints">['rotary_table_joint']</param> -->
-      <!-- <param name="command_interfaces">['position']</param> -->
-      <!-- <param name="state_interfaces">['position']</param> -->
-      <!-- Plain space-separated style (simplest) -->
-      <param name="joints">rotary_table_joint</param>
-      <param name="command_interfaces">position</param>
-      <param name="state_interfaces">position</param>
-      <param name="fake_sensor_commands">true</param>
-    </hardware>
-    <joint name="rotary_table_joint">
-      <state_interface   name="position"/>
-      <command_interface name="position"/>
-    </joint>
-  </ros2_control>
 </robot>

File: xarm_moveit_config/srdf/xarm_with_rotary_table.srdf.xacro (robot description, xacro)
@@ -1,4 +1,18 @@
 <?xml version="1.0" encoding="UTF-8"?>
-<robot name="XARM_WITH_ROTARY" xmlns="http://www.ros.org/schema/srdf" version="1.0">
+<robot
+  name="XARM_WITH_ROTARY"
+  xmlns="http://www.ros.org/schema/srdf"
+  xmlns:xacro="http://www.ros.org/wiki/xacro"
+  version="1.0">
+  <xacro:arg name="prefix" default="" />
+  <xacro:arg name="dof" default="7" />
+  <xacro:arg name="robot_type" default="xarm" />
+  <xacro:arg name="add_gripper" default="false"/>
+  <xacro:arg name="add_vacuum_gripper" default="false" />
+  <xacro:arg name="add_bio_gripper" default="false" />
+  <xacro:arg name="add_other_geometry" default="false" />
+  <xacro:include filename="$(find xarm_moveit_config)/srdf/xarm_macro.srdf.xacro" />
+  <xacro:xarm_macro_srdf prefix="$(arg prefix)" dof="$(arg dof)" robot_type="$(arg robot_type)"
+    add_gripper="$(arg add_gripper)" add_vacuum_gripper="$(arg add_vacuum_gripper)" add_bio_gripper="$(arg add_bio_gripper)" add_other_geometry="$(arg add_other_geometry)" />
   <!-- The full planning group -->
   <group name="xarm_with_rotary">
@@ -6,20 +20,12 @@
     <joint name="rotary_table_joint"/>
   </group>
-  <!-- For legacy compatibility, original xarm6 group -->
-  <group name="xarm6">
-    <chain base_link="link_base" tip_link="link_eef"/>
-  </group>
-  <!-- End effector -->
-  <end_effector name="xarm_gripper" parent_link="link_eef" group="xarm6"/>
   <!-- Virtual joints -->
-  <virtual_joint name="virtual_joint" type="fixed" parent_frame="world" child_link="link_base"/>
-  <!-- Disable collision checking for adjacent links -->
-  <disable_collisions link1="link_base" link2="link1" reason="Adjacent"/>
-  <disable_collisions link1="link1" link2="link2" reason="Adjacent"/>
-  <disable_collisions link1="link2" link2="link3" reason="Adjacent"/>
-  <disable_collisions link1="link3" link2="link4" reason="Adjacent"/>
-  <disable_collisions link1="link4" link2="link5" reason="Adjacent"/>
-  <disable_collisions link1="link5" link2="link6" reason="Adjacent"/>
-  <disable_collisions link1="link6" link2="link_eef" reason="Adjacent"/>
-  <disable_collisions link1="rotary_table_base" link2="rotary_plate" reason="Adjacent"/>
+  <virtual_joint name="virtual_joint" type="fixed" parent_frame="world" child_link="xarm_base"/>
+  <disable_collisions link1="rotary_table_base" link2="rotary_table_plate" reason="Adjacent"/>
+  <disable_collisions link1="rotary_table_base" link2="floor" reason="Adjacent"/>
+  <disable_collisions link1="xarm_base" link2="floor" reason="Adjacent"/>
+  <disable_collisions link1="xarm_base" link2="$(arg prefix)link_base" reason="Adjacent"/>
+  <disable_collisions link1="$(arg prefix)link1" link2="xarm_base" reason="Never"/>
+  <disable_collisions link1="$(arg prefix)link_base" link2="floor" reason="Never"/>
+  <disable_collisions link1="$(arg prefix)link1" link2="floor" reason="Never"/>
 </robot>
